File: pcb/p2000t-pico-web-interface.kicad_sch (KiCad schematic)
At the start: 21 parts, among them J1 P2000T Port 2, U1 74LVC273, U2 74HCT245, U3 74HCT245, U5 74LVC74, U6 74LVC08, U7 74HC32, U8 74HCT688, U9 74HCT138

Commit message: Removing diode from design, hardening interface
Parts:
- removed D1: 1N4148, Diode_THT:D_DO-35_SOD27_P7.62mm_Horizontal, symbol Diode:1N4148
Connections:
- no-connect marks 21 -> 22

Commit message: Adding LEDs to PCB
Parts:
- added D1: LED1, LED_THT:LED_D5.0mm, symbol Device:LED
- added D2: LED2, LED_THT:LED_D5.0mm, symbol Device:LED
- added R1, R2: 1k, Resistor_THT:R_Axial_DIN0207_L6.3mm_D2.5mm_P7.62mm_Horizontal, symbol Device:R
Connections:
- net GND: now also D1.1 (K), D2.1 (K)
- net LED1: now reaches A1.32 (GPIO27_ADC1)
- net LED1: now also R1.1
- net LED2: now reaches A1.34 (GPIO28_ADC2)
- net LED2: now also R2.1
- new net: D2.2 (A), R2.2
- new net: D1.2 (A), R1.2
- no-connect marks 22 -> 20
